Commit message: used xacro macros for wheel links for cleaner codes to the robot URDF

File: ros2_ws/src/my_robot_description/urdf/my_robot.urdf.xacro (robot description, xacro)
@@ -31,6 +31,7 @@
         </visual>
     </link>
-    <link name="right_rear_wheel_link">
-        <visual>
+    <xacro:macro name="wheel_link" params="prefix">
+        <link name="${prefix}_wheel_link">
+            <visual>
             <geometry>
                 <cylinder radius="${wheel_radius}" length="${wheel_length}" />
@@ -39,32 +40,10 @@
             <material name="yellow"/>
         </visual>
-    </link>
-    <link name="left_rear_wheel_link">
-        <visual>
-            <geometry>
-                <cylinder radius="0.1" length="0.05" />
-            </geometry>
-            <origin xyz="0.0 ${wheel_length} 0.0" rpy="${pi / 2.0} 0.0 0.0" />
-            <material name="yellow"/>
-        </visual>
-    </link>
-    <link name="right_front_wheel_link">
-        <visual>
-            <geometry>
-                <cylinder radius="0.1" length="0.05" />
-            </geometry>
-            <origin xyz="0.0 ${-wheel_length} 0.0" rpy="${pi / 2.0} 0.0 0.0" />
-            <material name="yellow"/>
-        </visual>
-    </link>
-    <link name="left_front_wheel_link">
-        <visual>
-            <geometry>
-                <cylinder radius="0.1" length="0.05" />
-            </geometry>
-            <origin xyz="0.0 ${wheel_length} 0.0" rpy="${pi / 2.0} 0.0 0.0" />
-            <material name="yellow"/>
-        </visual>
-    </link>
+        </link>
+    </xacro:macro>
+    <xacro:wheel_link prefix="right_rear"/>
+    <xacro:wheel_link prefix="right_front"/>
+    <xacro:wheel_link prefix="left_rear"/>
+    <xacro:wheel_link prefix="left_rear"/>
     <joint name="base_joint" type="fixed">
         <parent link = "base_footprint"/>
